File: Elektronik/Eagle/semesterprojekt.brd (EAGLE design)
At the start: 100 x 80 mm, 42 parts, among them T1 BC457, T2 BC457, T3 BC457, T4 BC457, T5 BC457, T6 BC457, T7 BC457, T8 BC457, T9 2N3565

Commit message: Boardv2
Parts:
- removed DRIVERX, DRIVERY, DRIVERZ, PLC-DRIVERX, PLC-DRIVERY, PLC-DRIVERZ: 22-23-2041, con-molex:22-23-2041
- removed PLC-SHARPENER: 22-23-2021, con-molex:22-23-2021
- removed R, R13, R17: 100k, rcl:0204/7
- removed R1, R12, R5: 2k, rcl:0204/7
- removed T4, T8: BC457, transistor:TO92
- removed T9: 2N3565, transistor:TO92
- added 24V, 24V-IN, PLC-SHARPENER-GND: 22-23-2021, con-molex:22-23-2021
- added 24V-OUT, DRIVER-X, DRIVER-Y, DRIVER-Z, PLC-X, PLC-Y, PLC-Z: 22-23-2031, con-molex:22-23-2031
- added D1: 1N4004, diode:DO41-10
- R14, R15, R16, R18, R19, R20: value 100k -> 5K
- moved R3 147.6 mm to (73.7, 16.5), turned to 270 degrees
- moved T2 127.2 mm to (61.0, 19.1)
- moved R4 125.5 mm to (71.1, 16.5), turned to 270 degrees
- moved R2 124.9 mm to (76.2, 16.5), turned to 270 degrees
- moved R20 123.8 mm to (64.8, 49.5), turned to 270 degrees
- moved T1 119.4 mm to (66.0, 25.4)
- moved R19 110.0 mm to (61.0, 49.5), turned to 270 degrees
- moved R18 96.1 mm to (57.1, 49.5), turned to 270 degrees
- moved R15 92.9 mm to (34.3, 50.8), turned to 270 degrees
- moved R10 92.2 mm to (26.7, 16.5), turned to 270 degrees
- moved T6 89.0 mm to (27.9, 31.8), turned to 270 degrees
- moved R8 85.2 mm to (39.4, 16.5), turned to 270 degrees
- moved R9 80.7 mm to (24.1, 16.5), turned to 270 degrees
- moved R7 78.4 mm to (41.9, 16.5), turned to 270 degrees
- moved R14 76.5 mm to (27.9, 50.8), turned to 270 degrees
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Connections:
- removed net N$16: SWITCH3+.1, SWITCH3+.2, SWITCH3+.3, T9.1
- removed net N$30: DRIVERX.1, R12.2
- removed net N$38: PLC-DRIVERX.1, R13.1
- removed net N$39: PLC-DRIVERX.3, R15.1
- removed net N$40: PLC-DRIVERX.4, R16.1
- removed net N$41: PLC-SWITCH.1, R.1
- removed net N$42: PLC-DRIVERY.3, R19.1
- removed net N$43: PLC-DRIVERY.4, R20.1
- removed net N$44: PLC-DRIVERY.2, R18.1
- removed net N$45: PLC-DRIVERY.1, R17.1
- net GND: now also 24V-IN.1, D1.C, PLC-SHARPENER-GND.2; no longer PLC-SHARPENER.2, SWITCH-GND.1, SWITCH-GND.2, SWITCH-GND.3, T4.3, T8.3, T9.3
- net N$1: now also 24V-IN.2, 24V-OUT.1, 24V-OUT.2, 24V-OUT.3; no longer DRIVERZ.1, R1.2
- net N$13: now also PLC-SHARPENER-GND.1; no longer PLC-SHARPENER.1
- net N$15: now also PLC-X.1, R16.1; no longer R13.2, T8.2
- net N$17: now also PLC-Y.3, R18.1; no longer R5.1, T4.1
- net N$19: now also DRIVER-Y.3; no longer DRIVERY.4
- net N$2: now also DRIVER-Z.1; no longer DRIVERZ.2
- net N$21: now also DRIVER-Y.2; no longer DRIVERY.3
- net N$23: now also DRIVER-Y.1; no longer DRIVERY.2
- net N$24: now also PLC-Y.2, R19.1; no longer DRIVERY.1, R5.2
- net N$26: now also DRIVER-X.2; no longer DRIVERX.3
- net N$29: now also PLC-Y.1, R20.1; no longer R12.1, T8.1
- net N$3: now also DRIVER-Z.2; no longer DRIVERZ.3
- net N$31: now also DRIVER-X.1; no longer DRIVERX.2
- net N$32: now also DRIVER-X.3; no longer DRIVERX.4
- net N$33: now also PLC-Z.1; no longer PLC-DRIVERZ.4
- net N$34: now also PLC-Z.2; no longer PLC-DRIVERZ.3
- net N$35: now also PLC-Z.3; no longer PLC-DRIVERZ.2
- net N$36: now also 24V.1, SWITCH3+.1, SWITCH3+.2, SWITCH3+.3; no longer PLC-DRIVERZ.1, R1.1
- net N$37: now also PLC-X.3; no longer PLC-DRIVERX.2
- net N$4: now also DRIVER-Z.3; no longer DRIVERZ.4
- net N$5: now also D1.A, PLC-SWITCH.1, SWITCH-GND.1, SWITCH-GND.2, SWITCH-GND.3; no longer R.2, T9.2
- net N$9: now also PLC-X.2, R15.1; no longer R17.2, T4.2
Routing:
- net N$10: track 0.00 -> 110.4 mm
- net N$8: track 0.00 -> 82.0 mm
- net N$36: track 0.00 -> 67.6 mm
- net N$5: track 0.00 -> 47.3 mm
- net N$18: track 0.00 -> 41.7 mm
- net N$29: track 0.00 -> 37.7 mm
- net N$13: track 0.00 -> 35.7 mm
- net N$1: track 0.00 -> 34.4 mm
- net N$22: track 0.00 -> 30.9 mm
- net N$7: track 0.00 -> 30.6 mm
- net N$24: track 0.00 -> 30.3 mm
- net N$33: track 0.00 -> 26.5 mm
- net N$11: track 0.00 -> 24.8 mm
- net N$20: track 0.00 -> 24.4 mm
- net N$14: track 0.00 -> 23.2 mm
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- added copper zone on layer 1, net GND
Other:
- board size 100 x 80 mm -> 84.8 x 80 mm
- board text added: "24V in"
- board text added: "24V out"
- board text added: "En-dir-step"
- board text added: "PLC-switch"
- board text added: "Sharp-6V"
- board text added: "Step-dir-en"
- board text added: "Switch end"
- board text added: "Switch start"

Commit message: Småændringer
Parts:
- removed 24V-OUT: 22-23-2031, con-molex:22-23-2031
- added X1: 22-23-2041, con-molex:22-23-2041
- renumbered PLC-SHARPENER-GND to PLC-24V
Connections:
- net N$1: now also X1.1, X1.2, X1.3, X1.4; no longer 24V-OUT.1, 24V-OUT.2, 24V-OUT.3
Routing:
- net N$5: track 47.3 -> 58.7 mm
- net N$1: track 34.4 -> 35.1 mm
- net N$13: track 35.7 -> 34.9 mm
Changed lines of the file:
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@@
 <elements>
 <element name="24V-&gt;6V" library="v-reg" library_urn="urn:adsk.eagle:library:409" package="78XXS" package3d_urn="urn:adsk.eagle:package:30342/1" value="" x="8.89" y="50.8" rot="R270"/>
-<element name="PLC-SHARPENER-GND" library="con-molex" library_urn="urn:adsk.eagle:library:165" package="22-23-2021" value="22-23-2021" x="20.32" y="72.39">
+<element name="PLC-24V" library="con-molex" library_urn="urn:adsk.eagle:library:165" package="22-23-2021" value="22-23-2021" x="20.32" y="72.39">
 <attribute name="MF" value="MOLEX" x="20.32" y="72.39" size="1.778" layer="27" display="off"/>
 <attribute name="MPN" value="22-23-2021" x="20.32" y="72.39" size="1.778" layer="27" display="off"/>
@@
 <element name="R3" library="rcl" library_urn="urn:adsk.eagle:library:334" package="0204/7" package3d_urn="urn:adsk.eagle:package:23498/1" value="2k" x="73.66" y="16.51" rot="R270"/>
 <element name="R4" library="rcl" library_urn="urn:adsk.eagle:library:334" package="0204/7" package3d_urn="urn:adsk.eagle:package:23498/1" value="2k" x="71.12" y="16.51" rot="R270"/>
-<element name="24V-OUT" library="con-molex" library_urn="urn:adsk.eagle:library:165" package="22-23-2031" value="22-23-2031" x="74.93" y="72.39">
-<attribute name="MF" value="MOLEX" x="74.93" y="72.39" size="1.778" layer="27" display="off"/>
-<attribute name="MPN" value="22-23-2031" x="74.93" y="72.39" size="1.778" layer="27" display="off"/>
-<attribute name="OC_FARNELL" value="1462950" x="74.93" y="72.39" size="1.778" layer="27" display="off"/>
-<attribute name="OC_NEWARK" value="30C0862" x="74.93" y="72.39" size="1.778" layer="27" display="off"/>
-</element>
 <element name="24V-IN" library="con-molex" library_urn="urn:adsk.eagle:library:165" package="22-23-2021" value="22-23-2021" x="74.93" y="50.8" rot="R270">
 <attribute name="MF" value="MOLEX" x="74.93" y="50.8" size="1.778" layer="27" rot="R270" display="off"/>
@@
 </element>
 <element name="D1" library="diode" library_urn="urn:adsk.eagle:library:210" package="DO41-10" package3d_urn="urn:adsk.eagle:package:43336/1" value="1N4004" x="11.43" y="26.162" rot="R180"/>
+<element name="X1" library="con-molex" library_urn="urn:adsk.eagle:library:165" package="22-23-2041" value="22-23-2041" x="74.93" y="71.12">
+<attribute name="MF" value="MOLEX" x="74.93" y="71.12" size="1.778" layer="27" display="off"/>
+<attribute name="MPN" value="22-23-2041" x="74.93" y="71.12" size="1.778" layer="27" display="off"/>
+<attribute name="OC_FARNELL" value="1462920" x="74.93" y="71.12" size="1.778" layer="27" display="off"/>
+<attribute name="OC_NEWARK" value="38C0355" x="74.93" y="71.12" size="1.778" layer="27" display="off"/>
+</element>
 </elements>
 <signals>
 <signal name="GND">
-<contactref element="PLC-SHARPENER-GND" pad="2"/>
+<contactref element="PLC-24V" pad="2"/>
 <contactref element="T3" pad="3"/>
 <contactref element="T2" pad="3"/>
@@
 </signal>
 <signal name="N$13">
-<contactref element="PLC-SHARPENER-GND" pad="1"/>
+<contactref element="PLC-24V" pad="1"/>
 <contactref element="24V-&gt;6V" pad="IN"/>
-<wire x1="19.05" y1="72.39" x2="19.05" y2="73.66" width="0.8128" layer="16"/>
-<wire x1="19.05" y1="73.66" x2="16.51" y2="76.2" width="0.8128" layer="16"/>
-<wire x1="16.51" y1="76.2" x2="10.16" y2="76.2" width="0.8128" layer="16"/>
-<wire x1="10.16" y1="76.2" x2="8.89" y2="74.93" width="0.8128" layer="16"/>
-<wire x1="8.89" y1="74.93" x2="8.89" y2="55.88" width="0.8128" layer="16"/>
-<wire x1="8.89" y1="55.88" x2="6.35" y2="53.34" width="0.8128" layer="16"/>
+<wire x1="19.05" y1="72.39" x2="15.24" y2="76.2" width="1.27" layer="16"/>
+<wire x1="15.24" y1="76.2" x2="10.16" y2="76.2" width="1.27" layer="16"/>
+<wire x1="10.16" y1="76.2" x2="8.89" y2="74.93" width="1.27" layer="16"/>
+<wire x1="8.89" y1="74.93" x2="8.89" y2="55.88" width="1.27" layer="16"/>
+<wire x1="8.89" y1="55.88" x2="6.35" y2="53.34" width="1.27" layer="16"/>
 </signal>
 <signal name="N$10">
@@
 <signal name="N$1">
 <contactref element="24V-IN" pad="2"/>
-<contactref element="24V-OUT" pad="1"/>
-<contactref element="24V-OUT" pad="2"/>
-<contactref element="24V-OUT" pad="3"/>
-<wire x1="74.93" y1="72.39" x2="74.93" y2="58.42" width="0.8128" layer="16"/>
-<wire x1="74.93" y1="58.42" x2="80.01" y2="53.34" width="0.8128" layer="16"/>
-<wire x1="80.01" y1="53.34" x2="80.01" y2="50.8" width="0.8128" layer="16"/>
-<wire x1="80.01" y1="50.8" x2="78.74" y2="49.53" width="0.8128" layer="16"/>
-<wire x1="78.74" y1="49.53" x2="74.93" y2="49.53" width="0.8128" layer="16"/>
-<wire x1="77.47" y1="72.39" x2="74.93" y2="72.39" width="0.8128" layer="16"/>
-<wire x1="72.39" y1="72.39" x2="74.93" y2="72.39" width="0.8128" layer="16"/>
+<contactref element="X1" pad="1"/>
+<contactref element="X1" pad="2"/>
+<contactref element="X1" pad="3"/>
+<contactref element="X1" pad="4"/>
+<wire x1="74.93" y1="49.53" x2="78.74" y2="49.53" width="1.27" layer="16"/>
+<wire x1="78.74" y1="49.53" x2="81.28" y2="52.07" width="1.27" layer="16"/>
+<wire x1="81.28" y1="52.07" x2="81.28" y2="68.58" width="1.27" layer="16"/>
+<wire x1="81.28" y1="68.58" x2="78.74" y2="71.12" width="1.27" layer="16"/>
+<wire x1="78.74" y1="71.12" x2="76.2" y2="71.12" width="1.27" layer="16"/>
+<wire x1="76.2" y1="71.12" x2="73.66" y2="71.12" width="1.27" layer="16"/>
+<wire x1="73.66" y1="71.12" x2="71.12" y2="71.12" width="1.27" layer="16"/>
 </signal>
 <signal name="N$9">
@@
 <wire x1="1.27" y1="58.42" x2="1.27" y2="30.48" width="0.8128" layer="16"/>
 <contactref element="PLC-SWITCH" pad="1"/>
-<wire x1="3.81" y1="60.96" x2="3.81" y2="72.39" width="0" layer="19" extent="16-16"/>
+<wire x1="3.81" y1="72.39" x2="3.81" y2="60.96" width="0.8128" layer="16"/>
 </signal>
 </signals>

Commit message: boardv4
Parts:
- removed 24V, 24V-IN, PLC-24V, PLC-SWITCH, SHARPENER: 22-23-2021, con-molex:22-23-2021
- removed D1: 1N4004, diode:DO41-10
- removed SWITCH-GND, SWITCH3+: 22-23-2031, con-molex:22-23-2031
- removed X1: 22-23-2041, con-molex:22-23-2041
- added R1, R12, R5: 5K, rcl:0204/7
- added SIGNAL-PLC, SPIDSER, VCC.-24V: 22-23-2021, con-molex:22-23-2021
- added SWITCH-X, SWITCH-Y, SWITCH-Z: 22-23-2031, con-molex:22-23-2031
- added T4, T8, T9: BC547, transistor:TO92
- DRIVER-X, DRIVER-Y, DRIVER-Z: value 22-23-2031 -> 22-23-2041; device con-molex:22-23-2031 -> con-molex:22-23-2041
- T1, T2, T3, T5, T6, T7: value BC457 -> BC547
- moved 24V->6V 42.7 mm to (25.4, 11.4)
- moved T3 39.1 mm to (57.1, 26.7), turned to 0 degrees
- moved PLC-Y 25.5 mm to (50.8, 47.0)
- moved R20 22.9 mm to (45.7, 36.8)
- moved R9 22.9 mm to (47.0, 15.2)
- moved R10 22.9 mm to (49.5, 15.2)
- moved R11 22.9 mm to (52.1, 15.2)
- moved T1 21.6 mm to (44.5, 26.7)
- moved DRIVER-X 21.6 mm to (48.3, 6.35)
- moved R7 20.4 mm to (62.2, 15.2)
- moved R8 20.4 mm to (59.7, 15.2)
- moved R6 20.4 mm to (64.8, 15.2)
- moved R16 19.8 mm to (26.7, 36.8)
- moved DRIVER-Y 19.1 mm to (61.0, 6.35)
- moved PLC-X 18.0 mm to (31.8, 47.0), turned to 0 degrees
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Connections:
- removed net N$1: 24V-IN.2, X1.1, X1.2, X1.3, X1.4
- removed net N$13: 24V->6V.IN, PLC-24V.1
- new net N$16: SIGNAL-PLC.1, SWITCH-X.2, SWITCH-Y.2, SWITCH-Z.2
- new net N$30: R3.1, T8.1
- new net N$38: R12.2, T4.2
- new net N$39: R5.2, T8.2
- new net N$40: R1.2, T9.2
- new net VCC: 24V->6V.IN, DRIVER-X.4, DRIVER-Y.4, DRIVER-Z.4, SWITCH-X.1, SWITCH-Y.1, SWITCH-Z.3, VCC.-24V.1
- net GND: now also SPIDSER.2, SWITCH-X.3, SWITCH-Y.3, SWITCH-Z.1, T4.3, T8.3, T9.3, VCC.-24V.2; no longer 24V-IN.1, D1.C, PLC-24V.2, SHARPENER.2
- net N$14: now also R4.1, T4.1; no longer 24V->6V.OUT, SHARPENER.1
- net N$33: now also R2.1, T9.1; no longer PLC-Z.1, R4.1
- net N$34: now also PLC-Z.1, R12.1; no longer PLC-Z.2, R3.1
- net N$35: now also PLC-Z.2, R5.1; no longer PLC-Z.3, R2.1
- net N$36: now also PLC-Z.3, R1.1; no longer 24V.1, SWITCH3+.1, SWITCH3+.2, SWITCH3+.3
- net N$5: now also 24V->6V.OUT, SPIDSER.1; no longer D1.A, PLC-SWITCH.1, SWITCH-GND.1, SWITCH-GND.2, SWITCH-GND.3
Routing:
- net VCC: track 0.00 -> 125.8 mm
- net N$10: track 110.4 -> 4.97 mm
- net N$8: track 82.0 -> 4.97 mm
- net N$36: track 67.6 -> 7.40 mm
- net N$16: track 0.00 -> 48.4 mm
- net N$5: track 58.7 -> 16.8 mm
- net N$1: track 35.1 -> 0.00 mm
- net N$13: track 34.9 -> 0.00 mm
- net N$29: track 37.7 -> 7.40 mm
- net N$7: track 30.6 -> 4.45 mm
- net N$18: track 41.7 -> 16.8 mm
- net N$24: track 30.3 -> 6.35 mm
- net N$22: track 30.9 -> 10.3 mm
- net N$11: track 24.8 -> 4.45 mm
- net N$33: track 26.5 -> 7.62 mm
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Other:
- board size 84.8 x 80 mm -> 87.3 x 57.1 mm
- board text added: "24v-signal-GND"
- board text added: "6V-GND"
- board text added: "GND-24V"
- board text added: "null-signal(sharp)"
- board text added: "step-dir-en"
- board text added: "step-dir-en-24v"
- board text removed: "24V in"
- board text removed: "24V out"
- board text removed: "En-dir-step"
- board text removed: "PLC-switch"
- board text removed: "Step-dir-en"
- board text removed: "Switch end"
- board text removed: "Switch start"
