File: Elektronik/Eagle/semesterprojekt.brd (EAGLE design)
At the start: 87.3 x 57.1 mm, 40 parts, among them T1 BC547, T2 BC547, T3 BC547, T4 BC547, T5 BC547, T6 BC547, T7 BC547, T8 BC547, T9 BC547

Commit message: PCB-2
Parts:
- added R13: 0, rcl:0204/7
- added U$1, U$2, U$3: (no value), holes:3,3
Connections:
- net GND: now also R13.1, R13.2
Routing:
- net GND: track 0.00 -> 26.5 mm
- net VCC: track 125.8 -> 122.6 mm
- net N$14: track 10.8 -> 13.8 mm
- net N$25: track 23.5 -> 26.5 mm
- net N$18: track 16.8 -> 19.7 mm
- net N$20: track 13.3 -> 16.1 mm
- net N$27: track 19.7 -> 22.5 mm
- net N$28: track 15.5 -> 18.3 mm
- net N$22: track 10.3 -> 12.7 mm
- net N$16: track 48.4 -> 47.3 mm
- net N$30: track 8.89 -> 9.94 mm
- added copper zone on layer 16, net GND
- removed copper zone on layer 1, net GND
Other:
- board text added: "GND-signal-24V"
- board text removed: "Sharp-6V"
