File: Elektronik/Eagle/semesterprojekt.sch (EAGLE design)
At the start: 42 parts, among them T1 BC457, T2 BC457, T3 BC457, T4 BC457, T5 BC457, T6 BC457, T7 BC457, T8 BC457, T9 2N3565

Commit message: Boardv2
Parts:
- removed DRIVERX, DRIVERY, DRIVERZ, PLC-DRIVERX, PLC-DRIVERY, PLC-DRIVERZ: 22-23-2041, con-molex:22-23-2041
- removed R, R13, R17: 100k, rcl:R-US_0204/7
- removed R1, R12, R5: 2k, rcl:R-US_0204/7
- removed T4, T8: BC457, transistor:2N3565
- removed T9: 2N3565, transistor:2N3565
- added 24V, 24V-IN: 22-23-2021, con-molex:22-23-2021
- added 24V-OUT, DRIVER-X, DRIVER-Y, DRIVER-Z, PLC-X, PLC-Y, PLC-Z: 22-23-2031, con-molex:22-23-2031
- added D1: 1N4004, diode:1N4004
- R14, R15, R16, R18, R19, R20: value 100k -> 5K
- renumbered PLC-SHARPENER to PLC-SHARPENER-GND
Connections:
- removed net N$16: SWITCH3+-1.S, SWITCH3+-2.S, SWITCH3+-3.S, T9.C
- removed net N$30: DRIVERX-1.S, R12.2
- removed net N$38: PLC-DRIVERX-1.S, R13.1
- removed net N$39: PLC-DRIVERX-3.S, R15.1
- removed net N$40: PLC-DRIVERX-4.S, R16.1
- removed net N$41: PLC-SWITCH-1.S, R.1
- removed net N$42: PLC-DRIVERY-3.S, R19.1
- removed net N$43: PLC-DRIVERY-4.S, R20.1
- removed net N$44: PLC-DRIVERY-2.S, R18.1
- removed net N$45: PLC-DRIVERY-1.S, R17.1
- net GND: now also 24V-IN-1.S, D1.C; no longer SWITCH-GND-1.S, SWITCH-GND-2.S, SWITCH-GND-3.S, T4.E, T8.E, T9.E
- net N$1: now also 24V-IN-2.S, 24V-OUT-1.S, 24V-OUT-2.S, 24V-OUT-3.S; no longer DRIVERZ-1.S, R1.2
- net N$15: now also PLC-X-1.S, R16.1; no longer R13.2, T8.B
- net N$17: now also PLC-Y-3.S, R18.1; no longer R5.1, T4.C
- net N$19: now also DRIVER-Y-3.S; no longer DRIVERY-4.S
- net N$2: now also DRIVER-Z-1.S; no longer DRIVERZ-2.S
- net N$21: now also DRIVER-Y-2.S; no longer DRIVERY-3.S
- net N$23: now also DRIVER-Y-1.S; no longer DRIVERY-2.S
- net N$24: now also PLC-Y-2.S, R19.1; no longer DRIVERY-1.S, R5.2
- net N$26: now also DRIVER-X-2.S; no longer DRIVERX-3.S
- net N$29: now also PLC-Y-1.S, R20.1; no longer R12.1, T8.C
- net N$3: now also DRIVER-Z-2.S; no longer DRIVERZ-3.S
- net N$31: now also DRIVER-X-1.S; no longer DRIVERX-2.S
- net N$32: now also DRIVER-X-3.S; no longer DRIVERX-4.S
- net N$33: now also PLC-Z-1.S; no longer PLC-DRIVERZ-4.S
- net N$34: now also PLC-Z-2.S; no longer PLC-DRIVERZ-3.S
- net N$35: now also PLC-Z-3.S; no longer PLC-DRIVERZ-2.S
- net N$36: now also 24V-1.S, SWITCH3+-1.S, SWITCH3+-2.S, SWITCH3+-3.S; no longer PLC-DRIVERZ-1.S, R1.1
- net N$37: now also PLC-X-3.S; no longer PLC-DRIVERX-2.S
- net N$4: now also DRIVER-Z-3.S; no longer DRIVERZ-4.S
- net N$5: now also D1.A, PLC-SWITCH-1.S, SWITCH-GND-1.S, SWITCH-GND-2.S, SWITCH-GND-3.S; no longer R.2, T9.B
- net N$9: now also PLC-X-2.S, R15.1; no longer R17.2, T4.B
Other:
- moved on the sheet: PLC-SWITCH-1, SWITCH-GND-1, SWITCH-GND-2, SWITCH-GND-3, SWITCH3+-1, SWITCH3+-2, SWITCH3+-3

Commit message: Småændringer
Parts:
- removed 24V-OUT: 22-23-2031, con-molex:22-23-2031
- added X1: 22-23-2041, con-molex:22-23-2041
- renumbered PLC-SHARPENER-GND to PLC-24V
Connections:
- net N$1: now also X1-1.S, X1-2.S, X1-3.S, X1-4.S; no longer 24V-OUT-1.S, 24V-OUT-2.S, 24V-OUT-3.S
Changed lines of the file:
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@@
 <part name="PLC-SWITCH" library="con-molex" library_urn="urn:adsk.eagle:library:165" deviceset="22-23-2021" device=""/>
 <part name="SWITCH3+" library="con-molex" library_urn="urn:adsk.eagle:library:165" deviceset="22-23-2031" device=""/>
-<part name="PLC-SHARPENER-GND" library="con-molex" library_urn="urn:adsk.eagle:library:165" deviceset="22-23-2021" device=""/>
+<part name="PLC-24V" library="con-molex" library_urn="urn:adsk.eagle:library:165" deviceset="22-23-2021" device=""/>
 <part name="GND10" library="supply1" library_urn="urn:adsk.eagle:library:371" deviceset="GND" device=""/>
 <part name="GND7" library="supply1" library_urn="urn:adsk.eagle:library:371" deviceset="GND" device=""/>
@@
 <part name="R4" library="rcl" library_urn="urn:adsk.eagle:library:334" deviceset="R-US_" device="0204/7" package3d_urn="urn:adsk.eagle:package:23498/1" value="2k"/>
 <part name="GND12" library="supply1" library_urn="urn:adsk.eagle:library:371" deviceset="GND" device=""/>
-<part name="24V-OUT" library="con-molex" library_urn="urn:adsk.eagle:library:165" deviceset="22-23-2031" device=""/>
 <part name="24V-IN" library="con-molex" library_urn="urn:adsk.eagle:library:165" deviceset="22-23-2021" device=""/>
 <part name="GND1" library="supply1" library_urn="urn:adsk.eagle:library:371" deviceset="GND" device=""/>
@@
 <part name="24V" library="con-molex" library_urn="urn:adsk.eagle:library:165" deviceset="22-23-2021" device=""/>
 <part name="D1" library="diode" library_urn="urn:adsk.eagle:library:210" deviceset="1N4004" device="" package3d_urn="urn:adsk.eagle:package:43336/1"/>
+<part name="X1" library="con-molex" library_urn="urn:adsk.eagle:library:165" deviceset="22-23-2041" device=""/>
 </parts>
 <sheets>
@@
 <instance part="SWITCH3+" gate="-2" x="0" y="124.46" rot="R90"/>
 <instance part="SWITCH3+" gate="-3" x="5.08" y="124.46" rot="R90"/>
-<instance part="PLC-SHARPENER-GND" gate="-1" x="-27.94" y="-40.64" rot="MR0"/>
-<instance part="PLC-SHARPENER-GND" gate="-2" x="-27.94" y="-43.18" rot="MR0"/>
+<instance part="PLC-24V" gate="-1" x="-27.94" y="-40.64" rot="MR0"/>
+<instance part="PLC-24V" gate="-2" x="-27.94" y="-43.18" rot="MR0"/>
 <instance part="GND10" gate="1" x="-17.78" y="-45.72"/>
 <instance part="GND7" gate="1" x="25.4" y="27.94"/>
@@
 <instance part="R4" gate="G$1" x="86.36" y="-10.16"/>
 <instance part="GND12" gate="1" x="114.3" y="-25.4"/>
-<instance part="24V-OUT" gate="-1" x="233.68" y="60.96"/>
-<instance part="24V-OUT" gate="-2" x="233.68" y="58.42"/>
-<instance part="24V-OUT" gate="-3" x="233.68" y="55.88"/>
 <instance part="24V-IN" gate="-1" x="180.34" y="60.96" rot="R180"/>
 <instance part="24V-IN" gate="-2" x="180.34" y="63.5" rot="R180"/>
@@
 <instance part="24V" gate="-1" x="-50.8" y="119.38" rot="R180"/>
 <instance part="D1" gate="1" x="22.86" y="104.14" rot="R270"/>
+<instance part="X1" gate="-1" x="233.68" y="60.96"/>
+<instance part="X1" gate="-2" x="233.68" y="58.42"/>
+<instance part="X1" gate="-3" x="233.68" y="55.88"/>
+<instance part="X1" gate="-4" x="233.68" y="53.34"/>
 </instances>
 <busses>
@@
 <net name="GND" class="0">
 <segment>
-<pinref part="PLC-SHARPENER-GND" gate="-2" pin="S"/>
+<pinref part="PLC-24V" gate="-2" pin="S"/>
 <pinref part="GND10" gate="1" pin="GND"/>
 <wire x1="-17.78" y1="-43.18" x2="-25.4" y2="-43.18" width="0.1524" layer="91"/>
@@
 <net name="N$13" class="0">
 <segment>
-<pinref part="PLC-SHARPENER-GND" gate="-1" pin="S"/>
+<pinref part="PLC-24V" gate="-1" pin="S"/>
 <wire x1="-25.4" y1="-40.64" x2="10.16" y2="-40.64" width="0.1524" layer="91"/>
 <pinref part="24V-&gt;6V" gate="1" pin="IN"/>
@@
 <wire x1="208.28" y1="58.42" x2="223.52" y2="58.42" width="0.1524" layer="91"/>
 <wire x1="223.52" y1="58.42" x2="223.52" y2="60.96" width="0.1524" layer="91"/>
-<pinref part="24V-OUT" gate="-1" pin="S"/>
 <wire x1="223.52" y1="60.96" x2="231.14" y2="60.96" width="0.1524" layer="91"/>
-<pinref part="24V-OUT" gate="-2" pin="S"/>
 <wire x1="223.52" y1="58.42" x2="231.14" y2="58.42" width="0.1524" layer="91"/>
-<pinref part="24V-OUT" gate="-3" pin="S"/>
 <wire x1="223.52" y1="58.42" x2="223.52" y2="55.88" width="0.1524" layer="91"/>
 <wire x1="223.52" y1="55.88" x2="231.14" y2="55.88" width="0.1524" layer="91"/>
@@
 <junction x="223.52" y="60.96"/>
 <junction x="223.52" y="55.88"/>
-</segment>
-</net>
+<pinref part="X1" gate="-1" pin="S"/>
+<pinref part="X1" gate="-2" pin="S"/>
+<pinref part="X1" gate="-3" pin="S"/>
+<pinref part="X1" gate="-4" pin="S"/>
+<wire x1="223.52" y1="55.88" x2="223.52" y2="53.34" width="0.1524" layer="91"/>
+<wire x1="223.52" y1="53.34" x2="231.14" y2="53.34" width="0.1524" layer="91"/>
+</segment>
+</net>

Commit message: boardv4
Parts:
- removed 24V, 24V-IN, PLC-24V, PLC-SWITCH, SHARPENER: 22-23-2021, con-molex:22-23-2021
- removed D1: 1N4004, diode:1N4004
- removed SWITCH-GND, SWITCH3+: 22-23-2031, con-molex:22-23-2031
- removed X1: 22-23-2041, con-molex:22-23-2041
- added R1, R12, R5: 5K, rcl:R-US_0204/7
- added SIGNAL-PLC, SPIDSER, VCC.-24V: 22-23-2021, con-molex:22-23-2021
- added SWITCH-X, SWITCH-Y, SWITCH-Z: 22-23-2031, con-molex:22-23-2031
- added T4, T8, T9: BC547, transistor:2N3565
- DRIVER-X, DRIVER-Y, DRIVER-Z: value 22-23-2031 -> 22-23-2041; device con-molex:22-23-2031 -> con-molex:22-23-2041
- T1, T2, T3, T5, T6, T7: value BC457 -> BC547
Connections:
- removed net N$1: 24V-IN-2.S, X1-1.S, X1-2.S, X1-3.S, X1-4.S
- removed net N$13: 24V->6V.IN, PLC-24V-1.S
- new net N$16: SIGNAL-PLC-1.S, SWITCH-X-2.S, SWITCH-Y-2.S, SWITCH-Z-2.S
- new net N$30: R3.1, T8.C
- new net N$38: R12.2, T4.B
- new net N$39: R5.2, T8.B
- new net N$40: R1.2, T9.B
- new net VCC: 24V->6V.IN, DRIVER-X-4.S, DRIVER-Y-4.S, DRIVER-Z-4.S, SWITCH-X-1.S, SWITCH-Y-1.S, SWITCH-Z-3.S, VCC.-24V-1.S
- net GND: now also SPIDSER-2.S, SWITCH-X-3.S, SWITCH-Y-3.S, SWITCH-Z-1.S, T4.E, T8.E, T9.E, VCC.-24V-2.S; no longer 24V-IN-1.S, D1.C, PLC-24V-2.S, SHARPENER-2.S
- net N$14: now also R4.1, T4.C; no longer 24V->6V.OUT, SHARPENER-1.S
- net N$33: now also R2.1, T9.C; no longer PLC-Z-1.S, R4.1
- net N$34: now also PLC-Z-1.S, R12.1; no longer PLC-Z-2.S, R3.1
- net N$35: now also PLC-Z-2.S, R5.1; no longer PLC-Z-3.S, R2.1
- net N$36: now also PLC-Z-3.S, R1.1; no longer 24V-1.S, SWITCH3+-1.S, SWITCH3+-2.S, SWITCH3+-3.S
- net N$5: now also 24V->6V.OUT, SPIDSER-1.S; no longer D1.A, PLC-SWITCH-1.S, SWITCH-GND-1.S, SWITCH-GND-2.S, SWITCH-GND-3.S
Other:
- moved on the sheet: 24V->6V, PLC-Z-1, PLC-Z-2, PLC-Z-3

Commit message: PCB-2
Parts:
- added R13: 0, rcl:R-US_0204/7
Connections:
- net GND: now also R13.1, R13.2
Changed lines of the file:
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@@
 <grid distance="0.1" unitdist="inch" unit="inch" style="lines" multiple="1" display="no" altdistance="0.01" altunitdist="inch" altunit="inch"/>
 <layers>
-<layer number="1" name="Top" color="4" fill="10" visible="no" active="no"/>
+<layer number="1" name="Top" color="4" fill="1" visible="no" active="no"/>
 <layer number="16" name="Bottom" color="1" fill="1" visible="no" active="no"/>
 <layer number="17" name="Pads" color="2" fill="1" visible="no" active="no"/>
 <layer number="18" name="Vias" color="2" fill="1" visible="no" active="no"/>
 <layer number="19" name="Unrouted" color="6" fill="1" visible="no" active="no"/>
-<layer number="20" name="Dimension" color="15" fill="1" visible="no" active="no"/>
+<layer number="20" name="Dimension" color="24" fill="1" visible="no" active="no"/>
 <layer number="21" name="tPlace" color="7" fill="1" visible="no" active="no"/>
 <layer number="22" name="bPlace" color="7" fill="1" visible="no" active="no"/>
@@
 <layer number="48" name="Document" color="7" fill="1" visible="no" active="no"/>
 <layer number="49" name="Reference" color="7" fill="1" visible="no" active="no"/>
-<layer number="51" name="tDocu" color="26" fill="1" visible="no" active="no"/>
+<layer number="51" name="tDocu" color="7" fill="1" visible="no" active="no"/>
 <layer number="52" name="bDocu" color="7" fill="1" visible="no" active="no"/>
 <layer number="90" name="Modules" color="5" fill="1" visible="yes" active="yes"/>
@@
 <part name="P+5" library="supply1" library_urn="urn:adsk.eagle:library:371" deviceset="VCC" device="" value="24V"/>
 <part name="P+6" library="supply1" library_urn="urn:adsk.eagle:library:371" deviceset="VCC" device="" value="24V"/>
+<part name="R13" library="rcl" library_urn="urn:adsk.eagle:library:334" deviceset="R-US_" device="0204/7" package3d_urn="urn:adsk.eagle:package:23498/1" value="0"/>
+<part name="GND12" library="supply1" library_urn="urn:adsk.eagle:library:371" deviceset="GND" device=""/>
+<part name="GND17" library="supply1" library_urn="urn:adsk.eagle:library:371" deviceset="GND" device=""/>
 </parts>
 <sheets>
@@
 <instance part="P+5" gate="VCC" x="111.76" y="20.32" rot="R90"/>
 <instance part="P+6" gate="VCC" x="111.76" y="53.34" rot="R90"/>
+<instance part="R13" gate="G$1" x="71.12" y="-30.48"/>
+<instance part="GND12" gate="1" x="63.5" y="-30.48" rot="R270"/>
+<instance part="GND17" gate="1" x="78.74" y="-30.48" rot="R90"/>
 </instances>
 <busses>
@@
 <pinref part="GND10" gate="1" pin="GND"/>
 </segment>
+<segment>
+<pinref part="R13" gate="G$1" pin="1"/>
+<pinref part="GND12" gate="1" pin="GND"/>
+</segment>
+<segment>
+<pinref part="R13" gate="G$1" pin="2"/>
+<pinref part="GND17" gate="1" pin="GND"/>
+</segment>
 </net>
