File: Elektronik/Stort kredslob.sch (EAGLE design)
At the start: 37 parts, among them T1 BC547, T2 BC547, T3 BC547, T4 BC547, T5 BC547, T6 BC547, T7 BC547, T8 BC547, T9 BC547

Commit message: Setup ændringer + lidt tekst
Connections:
- new net N$17: R4.1
Other:
- moved on the sheet: R1, R12, R13, R15, R18, R3, R4, R5, R6, R7, R9, T1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
