File: Elektronik/Switch-board.brd (EAGLE design)
At the start: 28.9 x 35.5 mm, 5 parts

Commit message: percentage virker
Parts:
- added U$1, U$2: (no value), holes:3,0
- moved Y 1.80 mm to (10.2, 17.8)
- moved PLC 1.27 mm to (22.9, 16.5)
- moved X 1.27 mm to (10.2, 6.35)
- moved Z 1.27 mm to (10.2, 30.5)
Routing:
- net GND: track 16.3 -> 18.3 mm
- net VCC: track 44.2 -> 43.0 mm
- net N$3: track 25.7 -> 24.4 mm
