File: Elektronik/Komplet elektronik kredsløb.sch (EAGLE design)
At the start: 47 parts, among them T1 BC547, T2 BC547, T3 BC547, T4 BC547, T5 BC547, T6 BC547, T7 BC547, T8 BC547, T9 BC547

Commit message: ff
Connections:
- net N$3: no longer Z-2.S
Changed lines of the file:
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@@
 <pinref part="PLC-X2" gate="A" pin="3"/>
 <wire x1="-7.62" y1="106.68" x2="-27.94" y2="106.68" width="0.1524" layer="91"/>
-<pinref part="Z" gate="-2" pin="S"/>
-<wire x1="-27.94" y1="106.68" x2="-27.94" y2="78.74" width="0.1524" layer="91"/>
-<wire x1="-27.94" y1="78.74" x2="-43.18" y2="78.74" width="0.1524" layer="91"/>
 </segment>
 </net>
